Commit message: Use model instead of package in xacro file

File: Tools/sitl_gazebo/models/F550/xacro/hexa_base.xacro (robot description, xacro)
@@ -23,5 +23,5 @@
         <origin xyz="0 0 0" rpy="0 0 0" />
         <geometry>
-          <mesh filename="package://F550/meshes/${mesh_file}"
+          <mesh filename="model://F550/meshes/${mesh_file}"
             scale="${mesh_scale}"/>
         </geometry>
@@ -88,5 +88,5 @@
       <visual>
         <geometry>
-          <mesh filename="package://F550/meshes/${wing_mesh_file}"
+          <mesh filename="model://F550/meshes/${wing_mesh_file}"
             scale="${wing_mesh_scale}"/>
         </geometry>
@@ -112,5 +112,5 @@
       <visual>
         <geometry>
-          <mesh filename="package://F550/meshes/${rotor_mesh_file}"
+          <mesh filename="model://F550/meshes/${rotor_mesh_file}"
             scale="${rotor_mesh_scale}"/>
         </geometry>
@@ -158,5 +158,5 @@
       <visual>
         <geometry>
-          <mesh filename="package://F550/meshes/${mesh_file}"
+          <mesh filename="model://F550/meshes/${mesh_file}"
             scale="${mesh_scale}" />
         </geometry>
