Commit message: Update URDF

File: Tools/sitl_gazebo/models/F550/F550.urdf (robot description, URDF)
Before this commit: robot F550, 17 links, 16 joints
Links:
- removed link fcu_px2
- removed link gps_here
- added link gps_holder; visual cylinder length=0.165 radius=0.002
- added link here_gps, mass 0.11416; visual mesh filename=package://F550/meshes/here_gps.STL scale=1 1 1
- added link pixhawk, mass 0.074008; visual mesh filename=package://F550/meshes/pixhawk.STL scale=1 1 1
- link wing_0: geometry visual mesh filename=package://F550/meshes/wing.STL scale=1 1 1
- link wing_1: geometry visual mesh filename=package://F550/meshes/wing.STL scale=1 1 1
- link wing_2: geometry visual mesh filename=package://F550/meshes/wing.STL scale=1 1 1
- link wing_3: geometry visual mesh filename=package://F550/meshes/wing.STL scale=1 1 1
- link wing_4: geometry visual mesh filename=package://F550/meshes/wing.STL scale=1 1 1
- link wing_5: geometry visual mesh filename=package://F550/meshes/wing.STL scale=1 1 1
Joints:
- removed joint fcu_px2_fix
- removed joint gps_here_fix
- added joint gps_holder_fix: type fixed, parent base_link, child gps_holder, origin xyz=0.1 0 0.08 rpy=0 0 0
- added joint here_gps_fix: type fixed, parent base_link, child here_gps, origin xyz=0.1 0 0.16 rpy=0 0 0, axis 0 0 0
- added joint pixhawk_fix: type fixed, parent base_link, child pixhawk, origin xyz=0 0 -0.04 rpy=0 0 0, axis 0 0 0
- joint rotor_0_joint: origin xyz=0.15910 -0.08203 0.059733 rpy=0 0 0 -> xyz=0.0865 0.0005 0.033 rpy=0 0 0
- joint rotor_1_joint: origin xyz=0.15910 0.15910 0.059733 rpy=0 0 0 -> xyz=0.0865 0.0005 0.033 rpy=0 0 0
- joint rotor_2_joint: origin xyz=0.15910 -0.08203 0.059733 rpy=0 0 0 -> xyz=0.0865 0.0005 0.033 rpy=0 0 0
- joint rotor_3_joint: origin xyz=0.15910 0.15910 0.059733 rpy=0 0 0 -> xyz=0.0865 0.0005 0.033 rpy=0 0 0
- joint rotor_4_joint: origin xyz=0.15910 0.15910 0.059733 rpy=0 0 0 -> xyz=0.0865 0.0005 0.033 rpy=0 0 0
- joint rotor_5_joint: origin xyz=0.15910 -0.08203 0.059733 rpy=0 0 0 -> xyz=0.0865 0.0005 0.033 rpy=0 0 0
- joint wing_0_joint: origin xyz=-0.21950 -0.17050 -0.04025 rpy=0 0 2.35619 -> xyz=0.1875 0 -0.0135 rpy=0 0 0
- joint wing_1_joint: origin xyz=0.04792 0 -0.04025 rpy=0 0 -0.78540 -> xyz=-0.1875 0 -0.0135 rpy=0 0 3.14159265359
- joint wing_2_joint: origin xyz=0.25843 -0.10426 -0.04025 rpy=0 0 -1.8326 -> xyz=-0.09375 0.16237976321 -0.0135 rpy=0 0 2.09439510239
- joint wing_3_joint: origin xyz=-0.02299 0.04331 -0.04025 rpy=0 0 1.30900 -> xyz=0.09375 -0.16237976321 -0.0135 rpy=0 0 -1.0471975512
- joint wing_4_joint: origin xyz=-0.02514 -0.04206 -0.04025 rpy=0 0 -2.87979 -> xyz=0.09375 0.16237976321 -0.0135 rpy=0 0 1.0471975512
- joint wing_5_joint: origin xyz=-0.03913 0.27481 -0.04025 rpy=0 0 0.261800 -> xyz=-0.09375 -0.16237976321 -0.0135 rpy=0 0 -2.09439510239

File: Tools/sitl_gazebo/models/F550_rd/F550_rd.urdf (robot description, URDF)
Before this commit: robot F550_rd, 19 links, 18 joints
Links:
- removed link fcu_px2
- removed link gps_here
- added link gps_holder; visual cylinder length=0.165 radius=0.002
- added link here_gps, mass 0.11416; visual mesh filename=package://F550/meshes/here_gps.STL scale=1 1 1
- added link pixhawk, mass 0.074008; visual mesh filename=package://F550/meshes/pixhawk.STL scale=1 1 1
- link wing_0: geometry visual mesh filename=package://F550/meshes/wing.STL scale=1 1 1
- link wing_1: geometry visual mesh filename=package://F550/meshes/wing.STL scale=1 1 1
- link wing_2: geometry visual mesh filename=package://F550/meshes/wing.STL scale=1 1 1
- link wing_3: geometry visual mesh filename=package://F550/meshes/wing.STL scale=1 1 1
- link wing_4: geometry visual mesh filename=package://F550/meshes/wing.STL scale=1 1 1
- link wing_5: geometry visual mesh filename=package://F550/meshes/wing.STL scale=1 1 1
Joints:
- removed joint fcu_px2_fix
- removed joint gps_here_fix
- added joint gps_holder_fix: type fixed, parent base_link, child gps_holder, origin xyz=0.1 0 0.08 rpy=0 0 0
- added joint here_gps_fix: type fixed, parent base_link, child here_gps, origin xyz=0.1 0 0.16 rpy=0 0 0, axis 0 0 0
- added joint pixhawk_fix: type fixed, parent base_link, child pixhawk, origin xyz=0 0 -0.04 rpy=0 0 0, axis 0 0 0
- joint rotor_0_joint: origin xyz=0.15910 -0.08203 0.059733 rpy=0 0 0 -> xyz=0.0865 0.0005 0.033 rpy=0 0 0
- joint rotor_1_joint: origin xyz=0.15910 0.15910 0.059733 rpy=0 0 0 -> xyz=0.0865 0.0005 0.033 rpy=0 0 0
- joint rotor_2_joint: origin xyz=0.15910 -0.08203 0.059733 rpy=0 0 0 -> xyz=0.0865 0.0005 0.033 rpy=0 0 0
- joint rotor_3_joint: origin xyz=0.15910 0.15910 0.059733 rpy=0 0 0 -> xyz=0.0865 0.0005 0.033 rpy=0 0 0
- joint rotor_4_joint: origin xyz=0.15910 0.15910 0.059733 rpy=0 0 0 -> xyz=0.0865 0.0005 0.033 rpy=0 0 0
- joint rotor_5_joint: origin xyz=0.15910 -0.08203 0.059733 rpy=0 0 0 -> xyz=0.0865 0.0005 0.033 rpy=0 0 0
- joint wing_0_joint: origin xyz=-0.21950 -0.17050 -0.04025 rpy=0 0 2.35619 -> xyz=0.1875 0 -0.0135 rpy=0 0 0
- joint wing_1_joint: origin xyz=0.04792 0 -0.04025 rpy=0 0 -0.78540 -> xyz=-0.1875 0 -0.0135 rpy=0 0 3.14159265359
- joint wing_2_joint: origin xyz=0.25843 -0.10426 -0.04025 rpy=0 0 -1.8326 -> xyz=-0.09375 0.16237976321 -0.0135 rpy=0 0 2.09439510239
- joint wing_3_joint: origin xyz=-0.02299 0.04331 -0.04025 rpy=0 0 1.30900 -> xyz=0.09375 -0.16237976321 -0.0135 rpy=0 0 -1.0471975512
- joint wing_4_joint: origin xyz=-0.02514 -0.04206 -0.04025 rpy=0 0 -2.87979 -> xyz=0.09375 0.16237976321 -0.0135 rpy=0 0 1.0471975512
- joint wing_5_joint: origin xyz=-0.03913 0.27481 -0.04025 rpy=0 0 0.261800 -> xyz=-0.09375 -0.16237976321 -0.0135 rpy=0 0 -2.09439510239

File: Tools/sitl_gazebo/models/F550_wireless/F550_wireless.urdf (robot description, URDF)
Before this commit: robot F550_wireless, 20 links, 19 joints
Links:
- removed link fcu_px2
- removed link gps_here
- added link gps_holder; visual cylinder length=0.165 radius=0.002
- added link here_gps, mass 0.11416; visual mesh filename=package://F550/meshes/here_gps.STL scale=1 1 1
- added link pixhawk, mass 0.074008; visual mesh filename=package://F550/meshes/pixhawk.STL scale=1 1 1
- link wing_0: geometry visual mesh filename=package://F550/meshes/wing.STL scale=1 1 1
- link wing_1: geometry visual mesh filename=package://F550/meshes/wing.STL scale=1 1 1
- link wing_2: geometry visual mesh filename=package://F550/meshes/wing.STL scale=1 1 1
- link wing_3: geometry visual mesh filename=package://F550/meshes/wing.STL scale=1 1 1
- link wing_4: geometry visual mesh filename=package://F550/meshes/wing.STL scale=1 1 1
- link wing_5: geometry visual mesh filename=package://F550/meshes/wing.STL scale=1 1 1
Joints:
- removed joint fcu_px2_fix
- removed joint gps_here_fix
- added joint gps_holder_fix: type fixed, parent base_link, child gps_holder, origin xyz=0.1 0 0.08 rpy=0 0 0
- added joint here_gps_fix: type fixed, parent base_link, child here_gps, origin xyz=0.1 0 0.16 rpy=0 0 0, axis 0 0 0
- added joint pixhawk_fix: type fixed, parent base_link, child pixhawk, origin xyz=0 0 -0.04 rpy=0 0 0, axis 0 0 0
- joint rotor_0_joint: origin xyz=0.15910 -0.08203 0.059733 rpy=0 0 0 -> xyz=0.0865 0.0005 0.033 rpy=0 0 0
- joint rotor_1_joint: origin xyz=0.15910 0.15910 0.059733 rpy=0 0 0 -> xyz=0.0865 0.0005 0.033 rpy=0 0 0
- joint rotor_2_joint: origin xyz=0.15910 -0.08203 0.059733 rpy=0 0 0 -> xyz=0.0865 0.0005 0.033 rpy=0 0 0
- joint rotor_3_joint: origin xyz=0.15910 0.15910 0.059733 rpy=0 0 0 -> xyz=0.0865 0.0005 0.033 rpy=0 0 0
- joint rotor_4_joint: origin xyz=0.15910 0.15910 0.059733 rpy=0 0 0 -> xyz=0.0865 0.0005 0.033 rpy=0 0 0
- joint rotor_5_joint: origin xyz=0.15910 -0.08203 0.059733 rpy=0 0 0 -> xyz=0.0865 0.0005 0.033 rpy=0 0 0
- joint wing_0_joint: origin xyz=-0.21950 -0.17050 -0.04025 rpy=0 0 2.35619 -> xyz=0.1875 0 -0.0135 rpy=0 0 0
- joint wing_1_joint: origin xyz=0.04792 0 -0.04025 rpy=0 0 -0.78540 -> xyz=-0.1875 0 -0.0135 rpy=0 0 3.14159265359
- joint wing_2_joint: origin xyz=0.25843 -0.10426 -0.04025 rpy=0 0 -1.8326 -> xyz=-0.09375 0.16237976321 -0.0135 rpy=0 0 2.09439510239
- joint wing_3_joint: origin xyz=-0.02299 0.04331 -0.04025 rpy=0 0 1.30900 -> xyz=0.09375 -0.16237976321 -0.0135 rpy=0 0 -1.0471975512
- joint wing_4_joint: origin xyz=-0.02514 -0.04206 -0.04025 rpy=0 0 -2.87979 -> xyz=0.09375 0.16237976321 -0.0135 rpy=0 0 1.0471975512
- joint wing_5_joint: origin xyz=-0.03913 0.27481 -0.04025 rpy=0 0 0.261800 -> xyz=-0.09375 -0.16237976321 -0.0135 rpy=0 0 -2.09439510239

Commit message: fix #2

File: Tools/sitl_gazebo/models/F550/F550.urdf (robot description, URDF)
Before this commit: robot F550, 18 links, 17 joints
Links:
- link here_gps: mass 0.11416 -> 0.045664
Joints:
- joint gps_holder_fix: origin xyz=0.1 0 0.08 rpy=0 0 0 -> xyz=0 -0.09 0.122 rpy=0 0 0
- joint here_gps_fix: origin xyz=0.1 0 0.16 rpy=0 0 0 -> xyz=0 -0.09 0.20 rpy=0 0 0
- joint pixhawk_fix: origin xyz=0 0 -0.04 rpy=0 0 0 -> xyz=0 0 0 rpy=0 0 0
- joint wing_0_joint: origin xyz=0.1875 0 -0.0135 rpy=0 0 0 -> xyz=0 -0.1875 0.026 rpy=0 0 -1.57079632679
- joint wing_1_joint: origin xyz=-0.1875 0 -0.0135 rpy=0 0 3.14159265359 -> xyz=0 0.1875 0.026 rpy=0 0 1.57079632679
- joint wing_2_joint: origin xyz=-0.09375 0.16237976321 -0.0135 rpy=0 0 2.09439510239 -> xyz=0.16237976321 0.09375 0.026 rpy=0 0 0.523598775598
- joint wing_3_joint: origin xyz=0.09375 -0.16237976321 -0.0135 rpy=0 0 -1.0471975512 -> xyz=-0.16237976321 -0.09375 0.026 rpy=0 0 -2.61799387799
- joint wing_4_joint: origin xyz=0.09375 0.16237976321 -0.0135 rpy=0 0 1.0471975512 -> xyz=0.16237976321 -0.09375 0.026 rpy=0 0 -0.523598775598
- joint wing_5_joint: origin xyz=-0.09375 -0.16237976321 -0.0135 rpy=0 0 -2.09439510239 -> xyz=-0.16237976321 0.09375 0.026 rpy=0 0 2.61799387799

File: Tools/sitl_gazebo/models/F550/xacro/F550_base.xacro (robot description, xacro)
@@ -15,14 +15,15 @@
   >
     <!-- units: kg･m^2 -->
-    <inertia ixx="0.0213982"
-             ixy="0"
-             ixz="0"
-             iyy="0.021956"
-             iyz="0.000340426"
-             izz="0.0398396"/>
+      <inertia
+        ixx="0.00012113"
+        ixy="-2.4623E-08"
+        ixz="1.6419E-06"
+        iyy="0.00013125"
+        iyz="6.0617E-07"
+        izz="1.8253E-05" />
   </xacro:property>
   <xacro:property name="collision_origin"
   >
-    <origin xyz="0 0 0" rpy="0 0 0" />
+    <origin xyz="0 0 0.03" rpy="0 0 0" />
   </xacro:property>
   <!-- rotors properties -->
@@ -137,6 +138,6 @@
     <!-- wing_origin -->
     <origin
-      xyz="0.1875 0 -0.0135"
-      rpy="0 0 0" />
+      xyz="0 -0.1875 0.026"
+      rpy="0 0 ${-pi / 2}" />
     <!-- wing_inertia_origin -->
     <xacro:insert_block name="wing_inertia_origin" />
@@ -178,6 +179,6 @@
     <!-- wing_origin -->
     <origin
-      xyz="-0.1875 0 -0.0135"
-      rpy="0 0 ${pi}" />
+      xyz="0 0.1875 0.026"
+      rpy="0 0 ${pi / 2}" />
     <!-- wing_inertia_origin -->
     <xacro:insert_block name="wing_inertia_origin" />
@@ -219,6 +220,6 @@
     <!-- wing_origin -->
     <origin
-      xyz="${0.1875 * cos(2*pi/3) } ${0.1875 * sin(2*pi/3)} -0.0135"
-      rpy="0 0 ${2*pi / 3}" />
+      xyz="${0.1875 * cos(pi/6)} ${0.1875 * sin(pi/6)} 0.026"
+      rpy="0 0 ${pi/6}" />
     <!-- wing_inertia_origin -->
     <xacro:insert_block name="wing_inertia_origin" />
@@ -260,6 +261,6 @@
     <!-- wing_origin -->
     <origin
-      xyz="${0.1875 * cos(-pi/3) } ${0.1875 * sin(-pi/3)} -0.0135"
-      rpy="0 0 ${ -pi / 3}" />
+      xyz="${0.1875 * cos(-5*pi/6)} ${0.1875 * sin(-5*pi/6)} 0.026"
+      rpy="0 0 ${-5*pi/6}" />
     <!-- wing_inertia_origin -->
     <xacro:insert_block name="wing_inertia_origin" />
@@ -301,6 +302,6 @@
     <!-- wing_origin -->
     <origin
-      xyz="${0.1875 * cos(pi/3) } ${0.1875 * sin(pi/3)} -0.0135"
-      rpy="0 0 ${ pi / 3}" />
+      xyz="${0.1875 * cos(-pi/6)} ${0.1875 * sin(-pi/6)} 0.026"
+      rpy="0 0 ${-pi/6}" />
     <!-- wing_inertia_origin -->
     <xacro:insert_block name="wing_inertia_origin" />
@@ -342,6 +343,6 @@
     <!-- wing_origin -->
     <origin
-      xyz="${0.1875 * cos(-2*pi/3) } ${0.1875 * sin(-2*pi/3)} -0.0135"
-      rpy="0 0 ${-2*pi / 3}" />
+      xyz="${0.1875 * cos(5*pi/6)} ${0.1875 * sin(5*pi/6)} 0.026"
+      rpy="0 0 ${5*pi/6}" />
     <!-- wing_inertia_origin -->
     <xacro:insert_block name="wing_inertia_origin" />
@@ -367,18 +368,18 @@
     <!-- ogigin -->
     <origin
-      xyz="0 0 -0.04"
+      xyz="0 0 0"
       rpy="0 0 0" />
     <!-- inertial origin -->
-      <origin
-        xyz="-9.4432E-05 -0.0024647 0.011865"
-        rpy="0 0 0" />
+    <origin
+      xyz="-0.0024647 9.4432E-05 0.011865"
+      rpy="0 0 0" />
     <!-- inertia -->
-      <inertia
-        ixx="3.8099E-06"
-        ixy="6.11E-09"
-        ixz="-7.5702E-08"
-        iyy="3.8198E-06"
-        iyz="2.3562E-07"
-        izz="4.7645E-08" />
+    <inertia
+      ixx="3.8198E-06"
+      ixy="-6.11E-09"
+      ixz="2.3562E-07"
+      iyy="3.8099E-06"
+      iyz="7.5702E-08"
+      izz="4.7645E-08" />
     <!-- axis -->
     <axis
@@ -388,5 +389,5 @@
   <xacro:accessory
     name="here_gps"
-    mass="0.11416"
+    mass="0.045664"
     mesh_file="here_gps.STL"
     mesh_scale="1 1 1"
@@ -396,18 +397,18 @@
     <!-- ogigin -->
     <origin
-      xyz="0.1 0 0.16"
+      xyz="0 -0.09 0.20"
       rpy="0 0 0" />
     <!-- inertial origin -->
     <origin
-      xyz="-1.3121E-06 -6.68E-05 0.0084082"
+      xyz="-6.68E-05 -0.0084082 1.31210000000051E-06"
       rpy="0 0 0" />
     <!-- inertia -->
     <inertia
-      ixx="2.98678228033835E-05"
-      ixy="-1.04111821878108E-10"
-      ixz="5.05387750838802E-11"
-      iyy="2.97244934804792E-05"
-      iyz="4.77263126398615E-08"
-      izz="5.59519257601009E-05" />
+      ixx="1.18897973921917E-05"
+      ixy="1.90905250559444E-08"
+      ixz="-4.16447287511186E-11"
+      iyy="2.23807703040404E-05"
+      iyz="2.02155100330627E-11"
+      izz="1.19471291213534E-05" />
     <!-- axis -->
     <axis
@@ -429,5 +430,5 @@
   <joint name="gps_holder_fix" type="fixed">
     <origin
-      xyz="0.1 0 0.08"
+      xyz="0 -0.09 0.122"
       rpy="0 0 0" />
     <parent link="base_link"/>

File: Tools/sitl_gazebo/models/F550_rd/F550_rd.urdf (robot description, URDF)
Before this commit: robot F550_rd, 20 links, 19 joints
Links:
- link here_gps: mass 0.11416 -> 0.045664
- link odroid_link: geometry visual mesh filename=package://F550_rd/meshes/odroid_xu4.STL scale=1 1 1
Joints:
- joint gps_holder_fix: origin xyz=0.1 0 0.08 rpy=0 0 0 -> xyz=0 -0.09 0.122 rpy=0 0 0
- joint here_gps_fix: origin xyz=0.1 0 0.16 rpy=0 0 0 -> xyz=0 -0.09 0.20 rpy=0 0 0
- joint lidar_joint: origin xyz=0 0.01 0.026 rpy=0 0 3.14 -> xyz=0.044 0 0.0655 rpy=0 0 0
- joint odoroid_joint: origin xyz=0 -0.032 0.038 rpy=0 0 1.57 -> xyz=-0.027 0 0.077 rpy=0 0 0
- joint pixhawk_fix: origin xyz=0 0 -0.04 rpy=0 0 0 -> xyz=0 0 0 rpy=0 0 0
- joint wing_0_joint: origin xyz=0.1875 0 -0.0135 rpy=0 0 0 -> xyz=0 -0.1875 0.026 rpy=0 0 -1.57079632679
- joint wing_1_joint: origin xyz=-0.1875 0 -0.0135 rpy=0 0 3.14159265359 -> xyz=0 0.1875 0.026 rpy=0 0 1.57079632679
- joint wing_2_joint: origin xyz=-0.09375 0.16237976321 -0.0135 rpy=0 0 2.09439510239 -> xyz=0.16237976321 0.09375 0.026 rpy=0 0 0.523598775598
- joint wing_3_joint: origin xyz=0.09375 -0.16237976321 -0.0135 rpy=0 0 -1.0471975512 -> xyz=-0.16237976321 -0.09375 0.026 rpy=0 0 -2.61799387799
- joint wing_4_joint: origin xyz=0.09375 0.16237976321 -0.0135 rpy=0 0 1.0471975512 -> xyz=0.16237976321 -0.09375 0.026 rpy=0 0 -0.523598775598
- joint wing_5_joint: origin xyz=-0.09375 -0.16237976321 -0.0135 rpy=0 0 -2.09439510239 -> xyz=-0.16237976321 0.09375 0.026 rpy=0 0 2.61799387799

File: Tools/sitl_gazebo/models/F550_rd/F550_rd.xacro (robot description, xacro)
@@ -24,5 +24,5 @@
   <!-- Joint -->
   <joint name="lidar_joint" type="revolute">
-    <origin xyz="0 0.01 0.026" rpy="0 0 3.14" />
+    <origin xyz="0.044 0 0.0655" rpy="0 0 0" />
     <child link="lidar_link"/>
     <parent link="base_link" />
@@ -33,5 +33,5 @@
     <material>Gazebo/DarkGrey</material>
     <sensor name="laser" type="ray">
-      <pose>0 -0.03 0.055 0 0 -1.57</pose>
+      <pose>0 0 0.055 0 0 0</pose>
       <ray>
         <scan>
@@ -78,7 +78,7 @@
     </inertial>
     <visual>
-      <origin xyz="0 0 0" rpy="3.14 0 0"/>
+      <origin xyz="0 0 0" rpy="0 0 0"/>
       <geometry>
-        <mesh filename="package://F550_rd/meshes/odroid.STL" scale="1 1 1"/>
+        <mesh filename="package://F550_rd/meshes/odroid_xu4.STL" scale="1 1 1"/>
       </geometry>
     </visual>
@@ -87,5 +87,5 @@
     <child link="odroid_link"/>
     <parent link="base_link"/>
-    <origin xyz="0 -0.032 0.038" rpy="0 0 1.57"/>
+    <origin xyz="-0.027 0 0.077" rpy="0 0 0"/>
   </joint>
   <gazebo reference="odroid_link">

File: Tools/sitl_gazebo/models/F550_wireless/F550_wireless.urdf (robot description, URDF)
Before this commit: robot F550_wireless, 21 links, 20 joints
Links:
- link here_gps: mass 0.11416 -> 0.045664
- link odroid_link: geometry visual mesh filename=package://F550_rd/meshes/odroid_xu4.STL scale=1 1 1
Joints:
- joint gps_holder_fix: origin xyz=0.1 0 0.08 rpy=0 0 0 -> xyz=0 -0.09 0.122 rpy=0 0 0
- joint here_gps_fix: origin xyz=0.1 0 0.16 rpy=0 0 0 -> xyz=0 -0.09 0.20 rpy=0 0 0
- joint lidar_joint: origin xyz=0 0.01 0.026 rpy=0 0 3.14 -> xyz=0.044 0 0.0655 rpy=0 0 0
- joint odoroid_joint: origin xyz=0 -0.032 0.038 rpy=0 0 1.57 -> xyz=-0.027 0 0.077 rpy=0 0 0
- joint pixhawk_fix: origin xyz=0 0 -0.04 rpy=0 0 0 -> xyz=0 0 0 rpy=0 0 0
- joint wing_0_joint: origin xyz=0.1875 0 -0.0135 rpy=0 0 0 -> xyz=0 -0.1875 0.026 rpy=0 0 -1.57079632679
- joint wing_1_joint: origin xyz=-0.1875 0 -0.0135 rpy=0 0 3.14159265359 -> xyz=0 0.1875 0.026 rpy=0 0 1.57079632679
- joint wing_2_joint: origin xyz=-0.09375 0.16237976321 -0.0135 rpy=0 0 2.09439510239 -> xyz=0.16237976321 0.09375 0.026 rpy=0 0 0.523598775598
- joint wing_3_joint: origin xyz=0.09375 -0.16237976321 -0.0135 rpy=0 0 -1.0471975512 -> xyz=-0.16237976321 -0.09375 0.026 rpy=0 0 -2.61799387799
- joint wing_4_joint: origin xyz=0.09375 0.16237976321 -0.0135 rpy=0 0 1.0471975512 -> xyz=0.16237976321 -0.09375 0.026 rpy=0 0 -0.523598775598
- joint wing_5_joint: origin xyz=-0.09375 -0.16237976321 -0.0135 rpy=0 0 -2.09439510239 -> xyz=-0.16237976321 0.09375 0.026 rpy=0 0 2.61799387799
